File: zglue-dragon-adapter.sch (KiCad schematic (older format))
At the start: 58 parts, among them J1 543630489, J2 543630489, U1 zGlue-Dragon

Commit message: Cleanup
Connections:
- net labels added: MIPI_SEL
Other:
- note added: "USB pullup"
- moved on the sheet: R11
Changed lines of the file:
@@
 encoding utf-8
 Sheet 1 1
-Title "zGlue Dragon Baseboard"
+Title "zGlue Dragon Adapter"
 Date ""
 Rev "1.0"
@@
 U 1 1 5D8F3A5B
 P 5100 3400
-F 0 "TP14" V 5100 3300 50  0000 C CNN
+F 0 "TP14" V 5100 3250 50  0000 C CNN
 F 1 "TP_SMD1MM" H 5100 3300 50  0001 C CNN
 F 2 "antmicro-footprints:Testpoint_smd_1mm" H 5300 3600 60  0001 L CNN
@@
 U 1 1 5D8F8F8D
 P 5100 3500
-F 0 "TP15" V 5100 3400 50  0000 C CNN
+F 0 "TP15" V 5100 3350 50  0000 C CNN
 F 1 "TP_SMD1MM" H 5100 3400 50  0001 C CNN
 F 2 "antmicro-footprints:Testpoint_smd_1mm" H 5300 3700 60  0001 L CNN
@@
 U 1 1 5D8F8FB7
 P 5100 3600
-F 0 "TP16" V 5100 3500 50  0000 C CNN
+F 0 "TP16" V 5100 3450 50  0000 C CNN
 F 1 "TP_SMD1MM" H 5100 3500 50  0001 C CNN
 F 2 "antmicro-footprints:Testpoint_smd_1mm" H 5300 3800 60  0001 L CNN
@@
 U 1 1 5D92F140
 P 5050 6250
-F 0 "TP13" V 5050 6150 50  0000 C CNN
+F 0 "TP13" V 5050 6100 50  0000 C CNN
 F 1 "TP_SMD1MM" H 5050 6150 50  0001 C CNN
 F 2 "antmicro-footprints:Testpoint_smd_1mm" H 5250 6450 60  0001 L CNN
@@
 U 1 1 5D935A2A
 P 5050 6150
-F 0 "TP12" V 5050 6050 50  0000 C CNN
+F 0 "TP12" V 5050 6000 50  0000 C CNN
 F 1 "TP_SMD1MM" H 5050 6050 50  0001 C CNN
 F 2 "antmicro-footprints:Testpoint_smd_1mm" H 5250 6350 60  0001 L CNN
@@
 U 1 1 5D9390AB
 P 5100 5650
-F 0 "TP17" V 5100 5550 50  0000 C CNN
+F 0 "TP17" V 5100 5500 50  0000 C CNN
 F 1 "TP_SMD1MM" H 5100 5550 50  0001 C CNN
 F 2 "antmicro-footprints:Testpoint_smd_1mm" H 5300 5850 60  0001 L CNN
@@
 U 1 1 5D971A5D
 P 1850 5800
-F 0 "TP9" V 1850 5700 50  0000 C CNN
+F 0 "TP9" V 1850 5650 50  0000 C CNN
 F 1 "TP_SMD1MM" H 1850 5700 50  0001 C CNN
 F 2 "antmicro-footprints:Testpoint_smd_1mm" H 2050 6000 60  0001 L CNN
@@
 U 1 1 5D971AC3
 P 1850 5900
-F 0 "TP10" V 1850 5800 50  0000 C CNN
+F 0 "TP10" V 1850 5750 50  0000 C CNN
 F 1 "TP_SMD1MM" H 1850 5800 50  0001 C CNN
 F 2 "antmicro-footprints:Testpoint_smd_1mm" H 2050 6100 60  0001 L CNN
@@
 U 1 1 5D971AF5
 P 1850 6000
-F 0 "TP11" V 1850 5900 50  0000 C CNN
+F 0 "TP11" V 1850 5850 50  0000 C CNN
 F 1 "TP_SMD1MM" H 1850 5900 50  0001 C CNN
 F 2 "antmicro-footprints:Testpoint_smd_1mm" H 2050 6200 60  0001 L CNN
@@
 Text Label 11100 2750 0    50   ~ 0
 DONE
-Text Label 6500 6500 0    50   ~ 0
+Text Label 9850 7950 0    50   ~ 0
 USB_DET
 Text Label 7900 3250 0    50   ~ 0
@@
 L antmicroResistors0402:R_1k5_0402 R11
 U 1 1 5DCE918C
-P 6300 6650
-F 0 "R11" V 6250 6400 60  0000 L CNN
-F 1 "R_1k5_0402" H 6300 6500 60  0001 C CNN
-F 2 "antmicro-footprints:0402-res" H 6500 6850 60  0001 L CNN
-F 3 "" H 6300 6650 50  0001 C CNN
-F 4 "PANASONIC_ELECTRONIC_COMPONENTS" H 6500 7050 60  0001 L CNN "Manufacturer"
-F 5 "ERJ2RKF1501X" H 6500 6950 60  0001 L CNN "MPN"
-F 6 "1k5" V 6350 6400 50  0000 L CNN "Val"
-	1    6300 6650
+P 9650 8100
+F 0 "R11" V 9600 7850 60  0000 L CNN
+F 1 "R_1k5_0402" H 9650 7950 60  0001 C CNN
+F 2 "antmicro-footprints:0402-res" H 9850 8300 60  0001 L CNN
+F 3 "" H 9650 8100 50  0001 C CNN
+F 4 "PANASONIC_ELECTRONIC_COMPONENTS" H 9850 8500 60  0001 L CNN "Manufacturer"
+F 5 "ERJ2RKF1501X" H 9850 8400 60  0001 L CNN "MPN"
+F 6 "1k5" V 9700 7850 50  0000 L CNN "Val"
+	1    9650 8100
 	0    1    1    0
 $EndComp
-Text Label 6500 6800 0    50   ~ 0
+Text Label 9850 8250 0    50   ~ 0
 USB_D_P
 Wire Wire Line
-	6300 6500 6850 6500
-Wire Wire Line
-	6300 6800 6850 6800
+	9650 7950 10200 7950
+Wire Wire Line
+	9650 8250 10200 8250
 Text Notes 8800 1400 0    50   ~ 0
 Mating - 556500488
@@
 Wire Wire Line
 	8750 6100 9700 6100
+Text Label 11100 3350 0    50   ~ 0
+PIO3
+Text Label 11100 3250 0    50   ~ 0
+PIO2
+Text Label 11100 3150 0    50   ~ 0
+PIO1
+Text Label 1950 2450 0    50   ~ 0
+MIPI_SEL
+Text Notes 9400 7550 0    79   ~ 16
+USB pullup
 $EndSCHEMATC
