File: zglue-dragon-adapter.kicad_pcb (KiCad board)
At the start: 6 copper layers, 25 x 20 mm, 59 parts, among them J1 543630489, J2 543630489, U1 zGlue-Dragon

Commit message: Library cleanup
Parts:
- C1, C10, C11, C12, C13, C14, C15, C2, C3, C4, C5, C6, C7, C8, C9: footprint antmicro-footprints:0402-cap -> zglue-dragon-adapter-footprints:0402-cap
- J1, J2: footprint antmicro-footprints:543630489 -> zglue-dragon-adapter-footprints:543630489
- R1, R10, R11, R12, R13, R14, R15, R16, R17, R18, R19, R2, R20, R21, R22, R23, R24, R25, R26, R3, R4, R5, R6, R7, R8, R9: footprint antmicro-footprints:0402-res -> zglue-dragon-adapter-footprints:0402-res
- TP1, TP10, TP11, TP12, TP14, TP15, TP16, TP17, TP2, TP3, TP4, TP5, TP7, TP8, TP9: footprint antmicro-footprints:Testpoint_smd_1mm -> zglue-dragon-adapter-footprints:Testpoint_smd_1mm
- U1: footprint lib:Z-Glue_LGA-96 -> zglue-dragon-adapter-footprints:Z-Glue_LGA-96
