File: zglue-gem1-adapter.sch (KiCad schematic (older format))
At the start: 59 parts, among them J1 543630489, J2 543630489, U1 zGlue-Dragon

Commit message: Updated naming convention, updated README
Parts:
- C1: symbol zglue-dragon-adapter:C_10u_0402 -> zglue-gem1-adapter:C_10u_0402
- C10, C11, C12, C14, C5, C6, C7, C8, C9: symbol zglue-dragon-adapter:C_100n_0402_6V3 -> zglue-gem1-adapter:C_100n_0402_6V3
- C13, C15: symbol zglue-dragon-adapter:C_10n_0402 -> zglue-gem1-adapter:C_10n_0402
- C2, C3, C4: symbol zglue-dragon-adapter:C_2u2_0402 -> zglue-gem1-adapter:C_2u2_0402
- J1, J2: symbol zglue-dragon-adapter:543630489 -> zglue-gem1-adapter:543630489
- R1, R15, R16, R17, R18, R19, R2, R20, R21, R22, R25, R26, R3, R4, R5, R6, R7, R8: symbol zglue-dragon-adapter:R_0R_0402 -> zglue-gem1-adapter:R_0R_0402
- R10, R12, R14, R23, R9: symbol zglue-dragon-adapter:R_100R_0402 -> zglue-gem1-adapter:R_100R_0402
- R11: symbol zglue-dragon-adapter:R_1k5_0402 -> zglue-gem1-adapter:R_1k5_0402
- R13: symbol zglue-dragon-adapter:R_10k_0402 -> zglue-gem1-adapter:R_10k_0402
- R24: symbol zglue-dragon-adapter:R_220R_0402 -> zglue-gem1-adapter:R_220R_0402
- TP1, TP10, TP11, TP12, TP14, TP15, TP16, TP17, TP2, TP3, TP4, TP5, TP7, TP8, TP9: symbol zglue-dragon-adapter:TP_SMD1MM -> zglue-gem1-adapter:TP_SMD1MM
- U1: value zGlue-Dragon -> zGlue-GEM1; symbol zglue-dragon-adapter:zGlue-Dragon -> zglue-gem1-adapter:zGlue-GEM1; MPN (none) -> GEM1; Manufacturer (none) -> zGlue/TSMC
Connections:
- wire segments 262 -> 255
Other:
- note added: "Configuration resistors"
- note added: "GEM1 chip"
- note added: "Place close to LGA Pads"
- note removed: "CSI INT"
- note removed: "Dragon chip"
- note removed: "MIPI termination"
- note removed: "Place close to zGlue pads"
- note removed: "USB pullup"
